Commit message: WBC for H1 done

File: models/robots/h1/h1.urdf (robot description, URDF)
Before this commit: robot h1_description, 27 links, 26 joints
Joints:
- joint left_foot: origin xyz=0 0 -0.076 rpy=0 1.57079633 0 -> xyz=0 0 -0.076 rpy=0 0 0
- joint right_foot: origin xyz=0 0 -0.076 rpy=0 1.57079633 0 -> xyz=0 0 -0.076 rpy=0 0 0
