Commit message: [in progress] Integrating GRT1 forWBC

File: models/robots/gr1/GR1T1.urdf (robot description, URDF)
Before this commit: robot GR1T1, 41 links, 40 joints
Links:
- removed link base
- added link left_foot_link, mass 1e-9
- added link left_hand_link, mass 1e-9
- added link right_foot_link, mass 1e-9
- added link right_hand_link, mass 1e-9
- added link torso_com_link, mass 1e-9
- added link torso_link, mass 6.45116957899581; collision box size=0.08 0.08 0.08; visual mesh filename=./meshes/base.STL
Joints:
- added joint left_foot: type fixed, parent l_foot_roll, child left_foot_link, origin xyz=0 0 -0.076 rpy=0 0 0
- added joint left_hand: type fixed, parent l_hand_pitch, child left_hand_link, origin xyz=0 0 0 rpy=0 0 0
- added joint right_foot: type fixed, parent r_foot_roll, child right_foot_link, origin xyz=0 0 -0.076 rpy=0 0 0
- added joint right_hand: type fixed, parent r_hand_pitch, child right_hand_link, origin xyz=0 0 0 rpy=0 0 0
- added joint torso_com: type fixed, parent torso_link, child torso_com_link, origin xyz=-0.0310745 -0.000497416 0.137484 rpy=0 0 0
- joint l_hip_roll: parent base -> torso_link
- joint r_hip_roll: parent base -> torso_link
- joint waist_pitch: axis 0 1 0 -> (none); limit lower=-0.52 upper=1.22 effort=33 velocity=6.28 -> (none); type revolute -> fixed
- joint waist_roll: axis 1 0 0 -> (none); limit lower=-0.7 upper=0.7 effort=33 velocity=6.28 -> (none); type revolute -> fixed
- joint waist_yaw: axis 0 0 1 -> (none); limit lower=-1.05 upper=1.05 effort=33 velocity=6.28 -> (none); parent base -> torso_link; type revolute -> fixed

Commit message: torso actuation

File: models/robots/gr1/GR1T1.urdf (robot description, URDF)
Before this commit: robot GR1T1, 46 links, 45 joints
Joints:
- joint waist_pitch: axis (none) -> 0 1 0; limit (none) -> lower=-0.52 upper=1.22 effort=33 velocity=6.28; type fixed -> revolute
- joint waist_roll: axis (none) -> 1 0 0; limit (none) -> lower=-0.7 upper=0.7 effort=33 velocity=6.28; type fixed -> revolute
- joint waist_yaw: axis (none) -> 0 0 1; limit (none) -> lower=-1.05 upper=1.05 effort=33 velocity=6.28; type fixed -> revolute
